Commit message: URDF

File: urdf/params.xacro (robot description, xacro)
@@ -7,18 +7,20 @@
   <xacro:property name="caster_diameter" value="0.04"/>
   <!-- Caster center to base edge -->
-  <xacro:property name="caster_inset" value="0.011"/>
+  <xacro:property name="caster_inset" value="0.031"/>
   <xacro:property name="floor_clearance" value="0.0169"/>
   <xacro:property name="base_diameter" value="0.34"/>
   <xacro:property name="wheel_base" value="0.286236"/>
-  <xacro:property name="lower_cylinder_height" value="0.032"/>
+  <xacro:property name="lower_cylinder_height" value="0.054"/>
   <xacro:property name="laser_puck_height" value="0.016"/>
   <xacro:property name="laser_puck_diameter" value="0.06"/>
-  <xacro:property name="laser_puck_offset" value="0.0384"/>
+  <!-- xacro:property name="laser_puck_z_offset" value="0.0384"/ -->
+  <xacro:property name="laser_puck_z_offset" value="0.008"/>
+  <xacro:property name="laser_puck_offset" value="0.01"/>
   <xacro:property name="laser_motor_diameter" value="0.02"/>
   <xacro:property name="lidar_motor_x_offset" value="0.04"/>
   <xacro:property name="lidar_motor_z_offset" value="0.012"/>
   <xacro:property name="laser_motor_height" value="0.01"/>
-  <xacro:property name="head_height" value="0.0388"/>
-  <xacro:property name="lidar_center_offset" value="0.000"/>
+  <!-- xacro:property name="head_height" value="0.0388"/ -->
+  <xacro:property name="lidar_center_x_offset" value="0.071047"/>
   <!-- N*m -->
   <xacro:property name="motor_stall_torque" value="0.171616375"/>

File: urdf/robot.urdf.xacro (robot description, xacro)
@@ -31,5 +31,5 @@
     <parent link="base_link"/>
     <child link="caster_link"/>
-    <origin xyz="${caster_inset-base_diameter/2} 0 ${caster_diameter/2-floor_clearance}" rpy="0 0 0"/>
+    <origin xyz="${-caster_inset+base_diameter/2} 0 ${caster_diameter/2-floor_clearance}" rpy="0 0 0"/>
   </joint>
   <link name="caster_link">
@@ -104,5 +104,5 @@
     <parent link="base_link"/>
     <child link="base_scan"/>
-    <origin xyz="${lidar_center_offset} 0 ${lower_cylinder_height + laser_puck_offset}" rpy="0 -${pi} 0"/>
+    <origin xyz="${lidar_center_x_offset} 0 ${lower_cylinder_height + laser_puck_z_offset}" rpy="0 -${pi} 0"/>
   </joint>
   <link name="base_scan">
@@ -143,5 +143,5 @@
     <xacro:solid_cylinder_inertia m="${laser_motor_mass}" r="${laser_motor_diameter/2}" h="${laser_motor_height}"/>
   </link>
-  <joint name="head_joint" type="fixed">
+  <!-- joint name="head_joint" type="fixed">
     <parent link="base_link"/>
     <child link="head_link"/>
@@ -163,4 +163,4 @@
     </collision>
     <xacro:solid_semi_ellipsoid_inertia m="${head_mass}" x="${base_diameter/2}" y="${base_diameter/2}" z="${head_height}"/>
-  </link>
+  </link -->
 </robot>
